File: LPC1114_LED_Cube.sch (KiCad schematic (older format))
At the start: 19 parts

Commit message: Created CH340T library and added to schematic
Parts:
- added U?: CH340T, Housings_SSOP:SSOP-20_5.3x7.2mm_Pitch0.65mm, symbol CH340T
- gave numbers to parts that had none: 1
Other:
- moved on the sheet: LAYER_VOUT
Changed lines of the file:
@@
 LIBS:audio
 LIBS:interface
+LIBS:ch340t
 EELAYER 25 0
 EELAYER END
@@
 	1800 900  2050 900
 $Comp
-L Conn_01x08 J?
+L Conn_01x08 LAYER_VOUT
 U 1 1 5B24F0DA
-P 9900 5150
-F 0 "J?" H 9900 5550 50  0000 C CNN
-F 1 "Conn_01x08" H 9900 4650 50  0000 C CNN
-F 2 "" H 9900 5150 50  0001 C CNN
-F 3 "" H 9900 5150 50  0001 C CNN
-	1    9900 5150
-	1    0    0    -1
-$EndComp
+P 10050 5400
+F 0 "LAYER_VOUT" H 10050 5800 50  0000 C CNN
+F 1 "Conn_01x08" H 10050 4900 50  0000 C CNN
+F 2 "" H 10050 5400 50  0001 C CNN
+F 3 "" H 10050 5400 50  0001 C CNN
+	1    10050 5400
+	1    0    0    -1
+$EndComp
+$Comp
+L CH340T U?
+U 1 1 5B2F3A76
+P 2000 5450
+F 0 "U?" H 2050 6200 60  0000 C CNN
+F 1 "CH340T" H 2050 5000 60  0000 C CNN
+F 2 "Housings_SSOP:SSOP-20_5.3x7.2mm_Pitch0.65mm" H 2000 5450 60  0001 C CNN
+F 3 "" H 2000 5450 60  0001 C CNN
+	1    2000 5450
+	1    0    0    -1
+$EndComp

Commit message: added USB-to-Serial bridge hardware added ld33v 3.3v voltage regulator
Parts:
- added C? (x2): 10uf, symbol CP1
- added C?: 22uf, symbol CP1
- added C?: 0.1uf, symbol C
- added C? (x2): 22pf, symbol C
- added J?: USB_A, symbol USB_A
- added U?: LD33V, symbol LD33V
- added Y?: 12MHZ, symbol Crystal
Connections:
- net labels added: CKO, RXD, TXD, V3, V5
- wire segments 47 -> 87
Other:
- moved on the sheet: LAYER_VOUT

Commit message: Added power and debug circuitry Started layer controller
Parts:
- added C? (x2): 22pf, symbol C
- added J?: Barrel_Jack, symbol Barrel_Jack
- added PWR_SEL: Conn_01x03, symbol Conn_01x03
- added SWDEBUG: Conn_02x05_Odd_Even, symbol Conn_02x05_Odd_Even
- added Y?: 12MHZ, symbol Crystal
- C? (x4): value C -> 0.1uf
Connections:
- net labels added: LAYER_0_ON, LAYER_1_ON, LAYER_2_ON, LAYER_3_ON, LAYER_4_ON, LAYER_5_ON, LAYER_6_ON, LAYER_7_ON, RXD_USB, SWCLK, SWDIO, TXD_USB, V5_AUX, V5_USB, _RESET
- net labels removed: RXD, TXD
- wire segments 87 -> 101
Other:
- moved on the sheet: C?, LAYER_VOUT

Commit message: Added AUX_SPI + Wireless Module Port Rearranged pins
Parts:
- added SPI/Wireless: Conn_02x04_Odd_Even, symbol Conn_02x04_Odd_Even
- C?: value C -> 0.1uf
Connections:
- net labels added: AUX_SPI_MISO, AUX_SPI_MOSI, AUX_SPI_SCK, AUX_SPI_SSEL, WIRELESS_CSN, WIRELESS_IRQ
- wire segments 101 -> 105
Changed lines of the file:
@@
 Text GLabel 5250 2850 2    60   Input ~ 0
 XERR_CH0
-Text GLabel 2750 2250 2    60   Output ~ 0
+Text GLabel 1350 2850 0    60   Output ~ 0
 BLANK
-Text GLabel 3450 2550 2    60   Input ~ 0
+Text GLabel 1350 3150 0    60   Output ~ 0
 DCPRG
 Text GLabel 1350 1550 0    60   Output ~ 0
@@
 Text GLabel 1350 2350 0    60   Output ~ 0
 LED_SIN
-Text GLabel 3450 2450 2    60   Input ~ 0
+Text GLabel 1350 2950 0    60   Output ~ 0
 VPRG
-Text GLabel 3450 2350 2    60   Input ~ 0
+Text GLabel 1350 2750 0    60   Output ~ 0
 XLAT
 Text GLabel 2750 2750 2    60   Input ~ 0
@@
 P 1650 900
 F 0 "C?" H 1675 1000 50  0000 L CNN
-F 1 "C" H 1675 800 50  0000 L CNN
+F 1 "0.1uf" H 1675 800 50  0000 L CNN
 F 2 "" H 1688 750 50  0001 C CNN
 F 3 "" H 1650 900 50  0001 C CNN
@@
 	1    0    0    -1
 $EndComp
-Text GLabel 4050 6600 2    60   Input ~ 0
+Text GLabel 4050 6600 2    60   BiDi ~ 0
 SWDIO
 Text GLabel 4050 6700 2    60   Input ~ 0
@@
 Text GLabel 5300 6300 2    60   Input ~ 0
 V5_AUX
-Text GLabel 6400 6300 0    60   Input ~ 0
+Text GLabel 6500 6100 0    60   Input ~ 0
 V5_USB
-Text GLabel 6400 6500 0    60   Input ~ 0
+Text GLabel 6500 6300 0    60   Input ~ 0
 V5_AUX
-Text GLabel 6400 6400 0    60   Output ~ 0
+Text GLabel 6500 6200 0    60   Output ~ 0
 V5
 Text GLabel 4950 7000 0    60   Input ~ 0
@@
 L Conn_01x03 PWR_SEL
 U 1 1 5B34D72E
-P 6600 6400
-F 0 "PWR_SEL" H 6600 6600 50  0000 C CNN
-F 1 "Conn_01x03" H 6600 6200 50  0000 C CNN
-F 2 "" H 6600 6400 50  0001 C CNN
-F 3 "" H 6600 6400 50  0001 C CNN
-	1    6600 6400
-	1    0    0    -1
-$EndComp
-Text GLabel 2750 1450 2    60   Output ~ 0
+P 6700 6200
+F 0 "PWR_SEL" H 6700 6400 50  0000 C CNN
+F 1 "Conn_01x03" H 6700 6000 50  0000 C CNN
+F 2 "" H 6700 6200 50  0001 C CNN
+F 3 "" H 6700 6200 50  0001 C CNN
+	1    6700 6200
+	1    0    0    -1
+$EndComp
+Text GLabel 2750 1850 2    60   Output ~ 0
 LAYER_0_ON
-Text GLabel 2750 1550 2    60   Output ~ 0
+Text GLabel 2750 1950 2    60   Output ~ 0
 LAYER_1_ON
-Text GLabel 2750 1650 2    60   Output ~ 0
+Text GLabel 2750 2050 2    60   Output ~ 0
 LAYER_2_ON
-Text GLabel 2750 1750 2    60   Output ~ 0
+Text GLabel 2750 2150 2    60   Output ~ 0
 LAYER_3_ON
-Text GLabel 2750 1850 2    60   Output ~ 0
+Text GLabel 2750 2250 2    60   Output ~ 0
 LAYER_4_ON
-Text GLabel 2750 1950 2    60   Output ~ 0
+Text GLabel 2750 2350 2    60   Output ~ 0
 LAYER_5_ON
-Text GLabel 2750 2050 2    60   Output ~ 0
+Text GLabel 2750 2450 2    60   Output ~ 0
 LAYER_6_ON
-Text GLabel 2750 2150 2    60   Output ~ 0
+Text GLabel 2750 2550 2    60   Output ~ 0
 LAYER_7_ON
 Text GLabel 9400 5150 0    60   Input ~ 0
@@
 F2 "LAYER_0" I L 9600 5150 60
 $EndSheet
+Text GLabel 2750 1550 2    60   Input ~ 0
+AUX_SPI_SCK
+Text GLabel 2750 1650 2    60   Input ~ 0
+AUX_SPI_MISO
+Text GLabel 2750 1750 2    60   Input ~ 0
+AUX_SPI_MOSI
+Text GLabel 2750 1450 2    60   Input ~ 0
+AUX_SPI_SSEL
+Text GLabel 8350 6150 0    60   Input ~ 0
+AUX_SPI_SSEL
+Text GLabel 8350 6250 0    60   Input ~ 0
+AUX_SPI_SCK
+Text GLabel 8350 6350 0    60   Input ~ 0
+AUX_SPI_MISO
+Text GLabel 8850 6250 2    60   Input ~ 0
+AUX_SPI_MOSI
+$Comp
+L Conn_02x04_Odd_Even SPI/Wireless
+U 1 1 5B361CD0
+P 8550 6150
+F 0 "SPI/Wireless" H 8600 6350 50  0000 C CNN
+F 1 "Conn_02x04_Odd_Even" H 8600 5850 50  0000 C CNN
+F 2 "" H 8550 6150 50  0001 C CNN
+F 3 "" H 8550 6150 50  0001 C CNN
+	1    8550 6150
+	1    0    0    -1
+$EndComp
+Text GLabel 8850 6050 2    60   Input ~ 0
+V3
+$Comp
+L GND #PWR?
+U 1 1 5B362960
+P 8000 5850
+F 0 "#PWR?" H 8000 5600 50  0001 C CNN
+F 1 "GND" H 8000 5700 50  0000 C CNN
+F 2 "" H 8000 5850 50  0001 C CNN
+F 3 "" H 8000 5850 50  0001 C CNN
+	1    8000 5850
+	1    0    0    -1
+$EndComp
+Text GLabel 8850 6150 2    60   Input ~ 0
+WIRELESS_CSN
+Text GLabel 8850 6350 2    60   Input ~ 0
+WIRELESS_IRQ
+Text GLabel 1350 3550 0    60   Input ~ 0
+WIRELESS_CSN
+Text GLabel 1350 3650 0    60   Input ~ 0
+WIRELESS_IRQ
+Wire Wire Line
+	8350 6050 8150 6050
+Wire Wire Line
+	8150 6050 8150 5800
+Wire Wire Line
+	8150 5800 8000 5800
+Wire Wire Line
+	8000 5800 8000 5850
 $EndSCHEMATC

Commit message: Finalized Schematic for Rev. A1
Parts:
- removed J?: USB_A, symbol USB_A
- added AUX_I/O_0: Conn_02x08_Top_Bottom, Connectors_Multicomp:Multicomp_MC9A12-1634_2x08x2.54mm_Straight, symbol Conn_02x08_Top_Bottom
- added C114: 10uf, Capacitors_THT:CP_Radial_D5.0mm_P2.50mm, symbol CP1
- added CH340_CKO_0: Conn_01x01, Pin_Headers:Pin_Header_Straight_1x01_Pitch2.54mm, symbol Conn_01x01
- added LED/SPI_0: Conn_01x04, Pin_Headers:Pin_Header_Straight_1x04_Pitch2.54mm, symbol Conn_01x04
- added USB_CONN_0: USB_B, Connectors:USB_B, symbol USB_B
- C101: renamed from C?; value 22uf -> 10uf; footprint (none) -> Capacitors_THT:CP_Radial_D5.0mm_P2.50mm
- C102, C103, C104, C105, C108, C109, C112, C113: renamed from C?; footprint (none) -> Capacitors_SMD:C_1206_HandSoldering
- C106, C107: renamed from C?; value 22pf -> 39pf; footprint (none) -> Capacitors_SMD:C_1206_HandSoldering
- C110, C111: renamed from C?; footprint (none) -> Capacitors_THT:CP_Radial_D5.0mm_P2.50mm
- LAYER_VOUT0: renamed from LAYER_VOUT; footprint (none) -> Pin_Headers:Pin_Header_Straight_1x08_Pitch2.54mm
- LED_CH0, LED_CH1, LED_CH2, LED_CH3: renamed from J?; footprint (none) -> Connectors_Multicomp:Multicomp_MC9A12-1634_2x08x2.54mm_Straight
- LED_CH0_CTRL0, LED_CH1_CTRL0, LED_CH2_CTRL0, LED_CH3_CTRL0: renamed from U?; footprint digikey-footprints:TSSOP-28-1EP_W4.40mm -> Housings_SSOP:TSSOP-28-1EP_4.4x9.7mm_Pitch0.65mm
- PWR_JACK0: renamed from J?; footprint (none) -> Connectors:BARREL_JACK
- PWR_SEL1: renamed from PWR_SEL; footprint (none) -> Pin_Headers:Pin_Header_Straight_1x03_Pitch2.54mm
- R101, R102, R103, R104: renamed from R?; footprint (none) -> Resistors_SMD:R_1206_HandSoldering
- SWDEBUG0: renamed from SWDEBUG; footprint (none) -> Pin_Headers:Pin_Header_Straight_2x05_Pitch1.27mm
- U105: renamed from U?; footprint (none) -> TO_SOT_Packages_THT:TO-220-3_Horizontal
- Wireless/SPI_1: renamed from SPI/Wireless; footprint (none) -> Pin_Headers:Pin_Header_Straight_2x04_Pitch2.54mm
- Y101, Y102: renamed from Y?; footprint (none) -> Crystals:Crystal_HC49-U_Vertical
- gave numbers to parts that had none: 2
Connections:
- net labels added: +5V, PIO0_11, PIO0_2, PIO0_3, PIO0_4, PIO0_5, PIO0_7, PIO0_8, PIO1_10, PIO1_11, PIO1_5, PIO3_4, PIO3_5
- net labels removed: CKO
- wire segments 105 -> 149
- no-connect marks 0 -> 14
Other:
- moved on the sheet: C102, C103, C104, C105, C106, C107, C108, C109, C112, C113, LAYER_VOUT0, LED_CH0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

Commit message: Initial PCB layout and some tracks Ingored more backup file types
Parts:
- removed AUX_I/O_0, LED_CH0, LED_CH1, LED_CH2, LED_CH3: Conn_02x08_Top_Bottom, Connectors_Multicomp:Multicomp_MC9A12-1634_2x08x2.54mm_Straight, symbol Conn_02x08_Top_Bottom
- added AUX_I/O_0, LED_CH0, LED_CH1, LED_CH2, LED_CH3: Conn_02x08_Odd_Even, Connectors_Multicomp:Multicomp_MC9A12-1634_2x08x2.54mm_Straight, symbol Conn_02x08_Odd_Even
- added ISP_ENTRY_SW0: SW_DIP_x01, Buttons_Switches_THT:SW_DIP_x1_W7.62mm_Slide, symbol SW_DIP_x01
- added RESET0: SW_SPST, Buttons_Switches_THT:SW_Tactile_Straight_KSA0Axx1LFTR, symbol SW_SPST
- LPC1114_0: footprint Package_QFP:LQFP-48_7x7mm_P0.5mm -> Housings_QFP:LQFP-48_7x7mm_Pitch0.5mm
- renumbered U105 to LD33V_0
Connections:
- net labels added: ISP_ENTRY
- wire segments 149 -> 157

Commit message: Fixed some schematic bugs. Added input mode switch.
Parts:
- removed ISP_ENTRY_SW0: SW_DIP_x01, Buttons_Switches_THT:SW_DIP_x1_W7.62mm_Slide, symbol SW_DIP_x01
- added MODE_SELECT_0: SW_DIP_x02, Buttons_Switches_THT:SW_DIP_x2_W7.62mm_Slide, symbol SW_DIP_x02
Connections:
- net labels added: INPUT_MODE_SELECT
- net labels removed: +3.3V
- wire segments 157 -> 164

Commit message: improved initial layout for better EMC and compactness Upgraded to KiCad 5.0
Parts:
- removed LED/SPI_0: Conn_01x04, Pin_Headers:Pin_Header_Straight_1x04_Pitch2.54mm, symbol Conn_01x04
- added XERR_CH0_BRIDGE0, XERR_CH0_BRIDGE1, XERR_CH1_BRIDGE0, XERR_CH1_BRIDGE1, XERR_CH2_BRIDGE0, XERR_CH2_BRIDGE1: Conn_01x01, Pin_Headers:Pin_Header_Straight_1x01_Pitch2.54mm, symbol conn:Conn_01x01
- added XERR_CH3_BRIDGE0: Conn_01x02, Pin_Headers:Pin_Header_Straight_1x02_Pitch2.54mm, symbol conn:Conn_01x02
- AUX_I/O_0, LED_CH0, LED_CH1, LED_CH2, LED_CH3: symbol Conn_02x08_Odd_Even -> conn:Conn_02x08_Odd_Even
- C101, C110, C111, C114: symbol CP1 -> Device:CP1
- C102, C103, C104, C105, C106, C107, C108, C109, C112, C113: symbol C -> Device:C
- CH340T_0: symbol CH340T -> ch340t:CH340T
- CH340_CKO_0: symbol Conn_01x01 -> conn:Conn_01x01
- LAYER_VOUT0: symbol Conn_01x08 -> conn:Conn_01x08
- LD33V_0: symbol LD33V -> ld33v:LD33V
- LED_CH0_CTRL0, LED_CH1_CTRL0, LED_CH2_CTRL0, LED_CH3_CTRL0: symbol TLC5940PWPR -> dk_PMIC-LED-Drivers:TLC5940PWPR
- LPC1114_0: symbol LPC1114FBD48-302 -> MCU_NXP_LPC:LPC1114FBD48-302
- MODE_SELECT_0: symbol SW_DIP_x02 -> Switch:SW_DIP_x02
- PWR_JACK0: symbol Barrel_Jack -> conn:Barrel_Jack
- PWR_SEL1: symbol Conn_01x03 -> conn:Conn_01x03
- R101, R102, R103, R104: symbol R -> Device:R
- RESET0: symbol SW_SPST -> Switch:SW_SPST
- SWDEBUG0: symbol Conn_02x05_Odd_Even -> conn:Conn_02x05_Odd_Even
- USB_CONN_0: symbol USB_B -> conn:USB_B
- Wireless/SPI_1: symbol Conn_02x04_Odd_Even -> conn:Conn_02x04_Odd_Even
- Y101, Y102: symbol Crystal -> Device:Crystal
Connections:
- net labels added: XERR_MCU_CH0, XERR_MCU_CH1, XERR_MCU_CH2, XERR_MCU_CH3
- wire segments 164 -> 193
