File: LPC1114_LED_Cube.kicad_pcb (KiCad board)
At the start: 2 copper layers, 100 x 100 mm, 80 parts, among them Q201 BSS138, Q202 BSS138, Q203 BSS138, Q204 BSS138, Q205 IRLML6402TRPBF, Q206 IRLML6402TRPBF, Q207 IRLML6402TRPBF, Q208 IRLML6402TRPBF, Q209 BSS138, Q210 BSS138, Q211 BSS138, Q212 BSS138, Q213 IRLML6402TRPBF, Q214 IRLML6402TRPBF, Q215 IRLML6402TRPBF, Q216 IRLML6402TRPBF, Y101 12MHZ, Y102 12MHZ

Commit message: more layout
Parts:
- added R217: 100R, Resistors_SMD:R_1206_HandSoldering, F.Cu at (102.2, 97.2)
- added R218: 100R, Resistors_SMD:R_1206_HandSoldering, F.Cu at (105.1, 97.2)
- added R219: 100R, Resistors_SMD:R_1206_HandSoldering, F.Cu at (108.0, 97.2)
- added R220: 100R, Resistors_SMD:R_1206_HandSoldering, F.Cu at (110.9, 97.2)
- added R221: 100R, Resistors_SMD:R_1206_HandSoldering, F.Cu at (113.7, 97.2)
- added R222: 100R, Resistors_SMD:R_1206_HandSoldering, F.Cu at (116.6, 97.2)
- added R223: 100R, Resistors_SMD:R_1206_HandSoldering, F.Cu at (119.5, 97.2)
- added R224: 100R, Resistors_SMD:R_1206_HandSoldering, F.Cu at (124.4, 95.1)
- moved C114 1.02 mm to (87.9, 105.5)
- moved C101 1.02 mm to (87.9, 97.9)
- moved C110 1.02 mm to (95.5, 105.5)
- moved C111 1.02 mm to (95.5, 97.9)
Connections:
- Q201 pad 1: LAYER_0_ON -> Net-(Q201-Pad1)
- Q202 pad 1: LAYER_1_ON -> Net-(Q202-Pad1)
- Q203 pad 1: LAYER_2_ON -> Net-(Q203-Pad1)
- Q204 pad 1: LAYER_3_ON -> Net-(Q204-Pad1)
- Q209 pad 1: LAYER_4_ON -> Net-(Q209-Pad1)
- Q210 pad 1: LAYER_5_ON -> Net-(Q210-Pad1)
- Q211 pad 1: LAYER_6_ON -> Net-(Q211-Pad1)
- Q212 pad 1: LAYER_7_ON -> Net-(Q212-Pad1)
- R209 pad 1: LAYER_0_ON -> Net-(Q201-Pad1)
- R210 pad 1: LAYER_1_ON -> Net-(Q202-Pad1)
- R211 pad 1: LAYER_2_ON -> Net-(Q203-Pad1)
- R212 pad 1: LAYER_3_ON -> Net-(Q204-Pad1)
- R213 pad 1: LAYER_4_ON -> Net-(Q209-Pad1)
- R214 pad 1: LAYER_5_ON -> Net-(Q210-Pad1)
- R215 pad 1: LAYER_6_ON -> Net-(Q211-Pad1)
- R216 pad 1: LAYER_7_ON -> Net-(Q212-Pad1)
Routing:
- net PIO0_11: track 0.00 -> 66.0 mm, vias 0 -> 4
- net RXD_USB: track 0.00 -> 65.9 mm, vias 0 -> 6
- net TXD_USB: track 0.00 -> 65.9 mm, vias 0 -> 6
- net _RESET: track 0.00 -> 65.8 mm, vias 0 -> 4
- net XERR_MCU_CH2: track 0.00 -> 65.5 mm, vias 0 -> 2
- net AUX_SPI_MOSI: track 0.00 -> 63.9 mm, vias 0 -> 2
- net PIO1_5: track 0.00 -> 60.1 mm, vias 0 -> 6
- net PIO1_11: track 0.00 -> 59.8 mm, vias 0 -> 6
- net AUX_SPI_SSEL: track 0.00 -> 59.1 mm, vias 0 -> 7
- net WIRELESS_CSN: track 0.00 -> 50.0 mm, vias 0 -> 4
- net INPUT_MODE_SELECT: track 0.00 -> 45.8 mm, vias 0 -> 2
- net WIRELESS_IRQ: track 0.00 -> 43.7 mm, vias 0 -> 2
- net XERR_MCU_CH3: track 0.00 -> 43.0 mm, vias 0 -> 2
- net VPRG: track 40.3 -> 81.3 mm, vias 6 -> 8
- net AUX_SPI_SCK: track 0.00 -> 39.6 mm, vias 0 -> 4
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
Commit message: Finished Rev 1A Layout
Routing:
- net V3: track 204.4 -> 437.0 mm, vias 10 -> 20
- net V5: track 78.1 -> 159.9 mm, vias 11 -> 12
- net AUX_SPI_MISO: track 0.00 -> 61.8 mm, vias 0 -> 2
- net PIO1_10: track 0.00 -> 60.1 mm, vias 0 -> 5
- net V5_USB: track 0.00 -> 49.6 mm
- net PIO0_8: track 0.00 -> 43.4 mm, vias 0 -> 4
- net SWCLK: track 0.00 -> 32.6 mm, vias 0 -> 2
- net GND: track 62.6 -> 92.4 mm, vias 51 -> 60
- net INPUT_MODE_SELECT: track 45.8 -> 67.7 mm, vias 2 -> 5
- net Net-(CH340T_0-Pad6): track 0.00 -> 17.7 mm
- net Net-(CH340T_0-Pad7): track 0.00 -> 14.8 mm
- net V5_AUX: track 0.00 -> 11.6 mm
- net Net-(CH340T_0-Pad1): track 0.00 -> 6.72 mm
- net PIO0_11: track 66.0 -> 68.1 mm
- net SWDIO: track 38.2 -> 39.3 mm
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Other:
- board text added: "100R"
- board text added: "10uF"
- board text added: "12.000MHZ XTAL 20PF"
- board text added: "1K"
- board text added: "ADDR_0 ADDR_63"
- board text added: "CSN"
- board text added: "CT00LPC111400CH340T00_R01AA_2018"
- board text added: "GND"
- board text added: "INPUT_MODE_SELECT"
- board text added: "IRQ"
- board text added: "LED Cube Controller Board ARM Cortex M0 (LPC1114) Rev 1A - Charles Trippe - Jul 29 2018"
- board text added: "LYR_0"
- board text added: "LYR_1"
- board text added: "LYR_2"
- board text added: "LYR_3"
- board text added: "LYR_4"
- board text added: "LYR_5"
- board text added: "LYR_6"
- board text added: "LYR_7"
- board text added: "MISO"
- board text added: "MOSI"
- board text added: "PIO0_11"
- board text added: "PIO0_3"
- board text added: "PIO0_4"
- board text added: "PIO0_5"
- board text added: "PIO0_8"
- board text added: "PIO1_10"
- board text added: "PIO1_11"
- board text added: "PIO1_5"
- board text added: "PIO3_4"
- board text added: "PIO3_5"
- board text added: "SCK"
- board text added: "SSEL"
- board text added: "V3"
- board text added: "V3+"
