File: LayerController.sch (KiCad schematic (older format))
At the start: 0 parts

Commit message: Finalized Schematic for Rev. A1
Parts:
- added Q201, Q202, Q203, Q204, Q209, Q210, Q211, Q212: BSS138, TO_SOT_Packages_SMD:SOT-23, symbol BSS138
- added Q205, Q206, Q207, Q208, Q213, Q214, Q215, Q216: IRLML6402TRPBF, TO_SOT_Packages_SMD:SOT-23, symbol IRLML6402TRPBF
- added R201, R202, R203, R204, R205, R206, R207, R208: 1K, Resistors_SMD:R_1206_HandSoldering, symbol R
Connections:
- net labels added: LAYER_1_ON, LAYER_1_PWR, LAYER_2_ON, LAYER_2_PWR, LAYER_3_ON, LAYER_3_PWR, LAYER_4_ON, LAYER_4_PWR, LAYER_5_ON, LAYER_5_PWR, LAYER_6_ON, LAYER_6_PWR, LAYER_7_ON, LAYER_7_PWR
- wire segments 0 -> 72

Commit message: improved initial layout for better EMC and compactness Upgraded to KiCad 5.0
Parts:
- added R209, R210, R211, R212, R213, R214, R215, R216: 1K, Resistors_SMD:R_1206_HandSoldering, symbol Device:R
- Q201, Q202, Q203, Q204, Q209, Q210, Q211, Q212: symbol BSS138 -> dk_Transistors-FETs-MOSFETs-Single:BSS138
- Q205, Q206, Q207, Q208, Q213, Q214, Q215, Q216: symbol IRLML6402TRPBF -> dk_Transistors-FETs-MOSFETs-Single:IRLML6402TRPBF
- R201, R202, R203, R204, R205, R206, R207, R208: symbol R -> Device:R
Connections:
- wire segments 72 -> 120

Commit message: more layout
Parts:
- added R217, R218, R219, R220, R221, R222, R223, R224: 100R, Resistors_SMD:R_1206_HandSoldering, symbol Device:R
Connections:
- wire segments 120 -> 128
Changed lines of the file:
@@
 Comment4 ""
 $EndDescr
-Text HLabel 2650 1850 0    60   Input ~ 0
+Text HLabel 2200 1850 0    60   Input ~ 0
 LAYER_0_ON
 Text GLabel 2950 1150 0    60   Input ~ 0
@@
 	1    0    0    1
 $EndComp
-Text HLabel 2650 3150 0    60   Input ~ 0
+Text HLabel 2200 3150 0    60   Input ~ 0
 LAYER_1_ON
 Text HLabel 4400 2950 2    60   Output ~ 0
 LAYER_1_PWR
-Text HLabel 2650 4400 0    60   Input ~ 0
+Text HLabel 2200 4400 0    60   Input ~ 0
 LAYER_2_ON
 Text HLabel 4400 4200 2    60   Output ~ 0
 LAYER_2_PWR
-Text HLabel 2650 5700 0    60   Input ~ 0
+Text HLabel 2200 5700 0    60   Input ~ 0
 LAYER_3_ON
 Text HLabel 4400 5500 2    60   Output ~ 0
 LAYER_3_PWR
-Text HLabel 5800 1900 0    60   Input ~ 0
+Text HLabel 5350 1900 0    60   Input ~ 0
 LAYER_4_ON
 Text HLabel 7550 1700 2    60   Output ~ 0
 LAYER_4_PWR
-Text HLabel 5800 3200 0    60   Input ~ 0
+Text HLabel 5350 3200 0    60   Input ~ 0
 LAYER_5_ON
 Text HLabel 7550 3000 2    60   Output ~ 0
 LAYER_5_PWR
-Text HLabel 5800 4450 0    60   Input ~ 0
+Text HLabel 5350 4450 0    60   Input ~ 0
 LAYER_6_ON
 Text HLabel 7550 4250 2    60   Output ~ 0
 LAYER_6_PWR
-Text HLabel 5800 5750 0    60   Input ~ 0
+Text HLabel 5350 5750 0    60   Input ~ 0
 LAYER_7_ON
 Text HLabel 7550 5550 2    60   Output ~ 0
@@
 	5950 1900 6050 1900
 Connection ~ 5950 1900
+$Comp
+L Device:R R217
+U 1 1 5B5EED1F
+P 2500 1850
+F 0 "R217" V 2580 1850 50  0000 C CNN
+F 1 "100R" V 2500 1850 50  0000 C CNN
+F 2 "Resistors_SMD:R_1206_HandSoldering" V 2430 1850 50  0001 C CNN
+F 3 "" H 2500 1850 50  0001 C CNN
+	1    2500 1850
+	0    1    1    0
+$EndComp
+Wire Wire Line
+	2350 1850 2200 1850
+$Comp
+L Device:R R218
+U 1 1 5B5FE9C5
+P 2500 3150
+F 0 "R218" V 2580 3150 50  0000 C CNN
+F 1 "100R" V 2500 3150 50  0000 C CNN
+F 2 "Resistors_SMD:R_1206_HandSoldering" V 2430 3150 50  0001 C CNN
+F 3 "" H 2500 3150 50  0001 C CNN
+	1    2500 3150
+	0    1    1    0
+$EndComp
+Wire Wire Line
+	2350 3150 2200 3150
+$Comp
+L Device:R R219
+U 1 1 5B602BCB
+P 2500 4400
+F 0 "R219" V 2580 4400 50  0000 C CNN
+F 1 "100R" V 2500 4400 50  0000 C CNN
+F 2 "Resistors_SMD:R_1206_HandSoldering" V 2430 4400 50  0001 C CNN
+F 3 "" H 2500 4400 50  0001 C CNN
+	1    2500 4400
+	0    1    1    0
+$EndComp
+Wire Wire Line
+	2350 4400 2200 4400
+$Comp
+L Device:R R220
+U 1 1 5B602BD2
+P 2500 5700
+F 0 "R220" V 2580 5700 50  0000 C CNN
+F 1 "100R" V 2500 5700 50  0000 C CNN
+F 2 "Resistors_SMD:R_1206_HandSoldering" V 2430 5700 50  0001 C CNN
+F 3 "" H 2500 5700 50  0001 C CNN
+	1    2500 5700
+	0    1    1    0
+$EndComp
+Wire Wire Line
+	2350 5700 2200 5700
+$Comp
+L Device:R R221
+U 1 1 5B60B355
+P 5650 1900
+F 0 "R221" V 5730 1900 50  0000 C CNN
+F 1 "100R" V 5650 1900 50  0000 C CNN
+F 2 "Resistors_SMD:R_1206_HandSoldering" V 5580 1900 50  0001 C CNN
+F 3 "" H 5650 1900 50  0001 C CNN
+	1    5650 1900
+	0    1    1    0
+$EndComp
+Wire Wire Line
+	5500 1900 5350 1900
+$Comp
+L Device:R R222
+U 1 1 5B60B35C
+P 5650 3200
+F 0 "R222" V 5730 3200 50  0000 C CNN
+F 1 "100R" V 5650 3200 50  0000 C CNN
+F 2 "Resistors_SMD:R_1206_HandSoldering" V 5580 3200 50  0001 C CNN
+F 3 "" H 5650 3200 50  0001 C CNN
+	1    5650 3200
+	0    1    1    0
+$EndComp
+Wire Wire Line
+	5500 3200 5350 3200
+$Comp
+L Device:R R223
+U 1 1 5B60B363
+P 5650 4450
+F 0 "R223" V 5730 4450 50  0000 C CNN
+F 1 "100R" V 5650 4450 50  0000 C CNN
+F 2 "Resistors_SMD:R_1206_HandSoldering" V 5580 4450 50  0001 C CNN
+F 3 "" H 5650 4450 50  0001 C CNN
+	1    5650 4450
+	0    1    1    0
+$EndComp
+Wire Wire Line
+	5500 4450 5350 4450
+$Comp
+L Device:R R224
+U 1 1 5B60B36A
+P 5650 5750
+F 0 "R224" V 5730 5750 50  0000 C CNN
+F 1 "100R" V 5650 5750 50  0000 C CNN
+F 2 "Resistors_SMD:R_1206_HandSoldering" V 5580 5750 50  0001 C CNN
+F 3 "" H 5650 5750 50  0001 C CNN
+	1    5650 5750
+	0    1    1    0
+$EndComp
+Wire Wire Line
+	5500 5750 5350 5750
 $EndSCHEMATC

Commit message: Rev 1B: Corrected silkscreen component values
Parts:
- R209, R210, R211, R212, R213, R214, R215, R216: value 1K -> 100K
Changed lines of the file:
@@
 P 2800 2000
 F 0 "R209" V 2880 2000 50  0000 C CNN
-F 1 "1K" V 2800 2000 50  0000 C CNN
+F 1 "100K" V 2800 2000 50  0000 C CNN
 F 2 "Resistors_SMD:R_1206_HandSoldering" V 2730 2000 50  0001 C CNN
 F 3 "" H 2800 2000 50  0001 C CNN
@@
 P 2800 3300
 F 0 "R210" V 2880 3300 50  0000 C CNN
-F 1 "1K" V 2800 3300 50  0000 C CNN
+F 1 "100K" V 2800 3300 50  0000 C CNN
 F 2 "Resistors_SMD:R_1206_HandSoldering" V 2730 3300 50  0001 C CNN
 F 3 "" H 2800 3300 50  0001 C CNN
@@
 P 2800 4550
 F 0 "R211" V 2880 4550 50  0000 C CNN
-F 1 "1K" V 2800 4550 50  0000 C CNN
+F 1 "100K" V 2800 4550 50  0000 C CNN
 F 2 "Resistors_SMD:R_1206_HandSoldering" V 2730 4550 50  0001 C CNN
 F 3 "" H 2800 4550 50  0001 C CNN
@@
 P 2800 5850
 F 0 "R212" V 2880 5850 50  0000 C CNN
-F 1 "1K" V 2800 5850 50  0000 C CNN
+F 1 "100K" V 2800 5850 50  0000 C CNN
 F 2 "Resistors_SMD:R_1206_HandSoldering" V 2730 5850 50  0001 C CNN
 F 3 "" H 2800 5850 50  0001 C CNN
@@
 P 5950 5900
 F 0 "R216" V 6030 5900 50  0000 C CNN
-F 1 "1K" V 5950 5900 50  0000 C CNN
+F 1 "100K" V 5950 5900 50  0000 C CNN
 F 2 "Resistors_SMD:R_1206_HandSoldering" V 5880 5900 50  0001 C CNN
 F 3 "" H 5950 5900 50  0001 C CNN
@@
 P 5950 4600
 F 0 "R215" V 6030 4600 50  0000 C CNN
-F 1 "1K" V 5950 4600 50  0000 C CNN
+F 1 "100K" V 5950 4600 50  0000 C CNN
 F 2 "Resistors_SMD:R_1206_HandSoldering" V 5880 4600 50  0001 C CNN
 F 3 "" H 5950 4600 50  0001 C CNN
@@
 P 5950 3350
 F 0 "R214" V 6030 3350 50  0000 C CNN
-F 1 "1K" V 5950 3350 50  0000 C CNN
+F 1 "100K" V 5950 3350 50  0000 C CNN
 F 2 "Resistors_SMD:R_1206_HandSoldering" V 5880 3350 50  0001 C CNN
 F 3 "" H 5950 3350 50  0001 C CNN
@@
 P 5950 2050
 F 0 "R213" V 6030 2050 50  0000 C CNN
-F 1 "1K" V 5950 2050 50  0000 C CNN
+F 1 "100K" V 5950 2050 50  0000 C CNN
 F 2 "Resistors_SMD:R_1206_HandSoldering" V 5880 2050 50  0001 C CNN
 F 3 "" H 5950 2050 50  0001 C CNN
